Commit message: moveit_fixes

File: ceeorobot_control/urdf/ceeorobot_controlled.urdf.xacro (robot description, xacro)
@@ -45,5 +45,5 @@
   <!--If you had more controlled devices in your description, e.g. a gripper, you can add another ros2_control tag here-->
   <xacro:robotiq_hande_ros2_control
-      prefix="${ur_type}_"
+      prefix=""
       parent="${ur_type}_tool0"
       name="handE"

File: ceeorobot_description/urdf/ceeorobot_cell_macro.xacro (robot description, xacro)
@@ -17,14 +17,18 @@
       <child link="table" />
     </joint>
-    <link name="table">
+  <link name="table">
       <visual>
         <geometry>
+          <mesh filename="package://ceeorobot_description/meshes/fzi_table.dae"/>
         </geometry>
         <origin rpy="0 0 0" xyz="0.75 0.5 -1"/>
       </visual>
+      <collision>
+        <geometry>
+          <mesh filename="package://ceeorobot_description/meshes/fzi_table.dae"/>
+        </geometry>
+        <origin rpy="0 0 0" xyz="0.75 0.5 -1"/>
+      </collision>
     </link>
-    <material name="white">
-      <color rgba="1 1 1 1"/>
-    </material>
     <link name="robot_mount"/>
     <joint name="base_to_robot_mount" type="fixed">
