Commit message: flat version for use with springcontroller

File: ceeorobot_description/urdf/ceeorobot_flat.urdf (robot description, URDF)
Before this commit: robot ceeorobot, 20 links, 19 joints
Links:
- removed link robotiq_hande_coupler
- removed link robotiq_hande_end
- removed link robotiq_hande_left_finger
- removed link robotiq_hande_link
- removed link robotiq_hande_right_finger
Joints:
- removed joint robotiq_hande_base_joint
- removed joint robotiq_hande_coupler_joint
- removed joint robotiq_hande_end_joint
- removed joint robotiq_hande_left_finger_joint
- removed joint robotiq_hande_right_finger_joint
- joint table_base_joint: origin xyz=0 0 1 rpy=0 0 0 -> xyz=0 0 0 rpy=0 0 0

Commit message: fixed flat config to use ur3e prefix

File: ceeorobot_description/urdf/ceeorobot_flat.urdf (robot description, URDF)
Before this commit: robot ceeorobot, 15 links, 14 joints
Links:
- removed link ur3_base
- removed link ur3_base_link
- removed link ur3_base_link_inertia
- removed link ur3_flange
- removed link ur3_forearm_link
- removed link ur3_ft_frame
- removed link ur3_shoulder_link
- removed link ur3_tool0
- removed link ur3_upper_arm_link
- removed link ur3_wrist_1_link
- removed link ur3_wrist_2_link
- removed link ur3_wrist_3_link
- added link ur3e_base
- added link ur3e_base_link
- added link ur3e_base_link_inertia, mass 2.0; collision mesh filename=file:///home/kat/workspace/src/ceeorobot_cell/ceeorobot_des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; visual mesh filename=file:///home/kat/workspace/src/ceeorobot_cell/ceeorobot_des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
- added link ur3e_flange
- added link ur3e_forearm_link, mass 1.26; collision mesh filename=file:///home/kat/workspace/src/ceeorobot_cell/ceeorobot_des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; visual mesh filename=file:///home/kat/workspace/src/ceeorobot_cell/ceeorobot_des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
- added link ur3e_ft_frame
- added link ur3e_shoulder_link, mass 2.0; collision mesh filename=file:///home/kat/workspace/src/ceeorobot_cell/ceeorobot_des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; visual mesh filename=file:///home/kat/workspace/src/ceeorobot_cell/ceeorobot_des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
- added link ur3e_tool0
- added link ur3e_upper_arm_link, mass 3.42; collision mesh filename=file:///home/kat/workspace/src/ceeorobot_cell/ceeorobot_des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; visual mesh filename=file:///home/kat/workspace/src/ceeorobot_cell/ceeorobot_des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
- added link ur3e_wrist_1_link, mass 0.8; collision mesh filename=file:///home/kat/workspace/src/ceeorobot_cell/ceeorobot_des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; visual mesh filename=file:///home/kat/workspace/src/ceeorobot_cell/ceeorobot_des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
- added link ur3e_wrist_2_link, mass 0.8; collision mesh filename=file:///home/kat/workspace/src/ceeorobot_cell/ceeorobot_des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; visual mesh filename=file:///home/kat/workspace/src/ceeorobot_cell/ceeorobot_des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
- added link ur3e_wrist_3_link, mass 0.35; collision mesh filename=file:///home/kat/workspace/src/ceeorobot_cell/ceeorobot_des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; visual mesh filename=file:///home/kat/workspace/src/ceeorobot_cell/ceeorobot_des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
Joints:
- removed joint ur3_base_joint
- removed joint ur3_base_link-base_fixed_joint
- removed joint ur3_base_link-base_link_inertia
- removed joint ur3_elbow_joint
- removed joint ur3_flange-tool0
- removed joint ur3_shoulder_lift_joint
- removed joint ur3_shoulder_pan_joint
- removed joint ur3_wrist_1_joint
- removed joint ur3_wrist_2_joint
- removed joint ur3_wrist_3-flange
- removed joint ur3_wrist_3_joint
- removed joint ur3_wrist_3_link-ft_frame
- added joint ur3e_base_joint: type fixed, parent robot_mount, child ur3e_base_link, origin xyz=0 0 0 rpy=0 0 0
- added joint ur3e_base_link-base_fixed_joint: type fixed, parent ur3e_base_link, child ur3e_base, origin xyz=0 0 0 rpy=0 0 3.141592653589793
- added joint ur3e_base_link-base_link_inertia: type fixed, parent ur3e_base_link, child ur3e_base_link_inertia, origin xyz=0 0 0 rpy=0 0 3.141592653589793
- added joint ur3e_elbow_joint: type revolute, parent ur3e_upper_arm_link, child ur3e_forearm_link, origin xyz=-0.24365 0 0 rpy=0 0 0, axis 0 0 1, limit lower=-3.141592653589793 upper=3.141592653589793 effort=28.0 velocity=3.141592653589793
- added joint ur3e_flange-tool0: type fixed, parent ur3e_flange, child ur3e_tool0, origin xyz=0 0 0 rpy=1.5707963267948966 0 1.5707963267948966
- added joint ur3e_shoulder_lift_joint: type revolute, parent ur3e_shoulder_link, child ur3e_upper_arm_link, origin xyz=0 0 0 rpy=1.570796327 0 0, axis 0 0 1, limit lower=-6.283185307179586 upper=6.283185307179586 effort=56.0 velocity=3.141592653589793
- added joint ur3e_shoulder_pan_joint: type revolute, parent ur3e_base_link_inertia, child ur3e_shoulder_link, origin xyz=0 0 0.1519 rpy=0 0 0, axis 0 0 1, limit lower=-6.283185307179586 upper=6.283185307179586 effort=56.0 velocity=3.141592653589793
- added joint ur3e_wrist_1_joint: type revolute, parent ur3e_forearm_link, child ur3e_wrist_1_link, origin xyz=-0.21325 0 0.11235 rpy=0 0 0, axis 0 0 1, limit lower=-6.283185307179586 upper=6.283185307179586 effort=12.0 velocity=6.283185307179586
- added joint ur3e_wrist_2_joint: type revolute, parent ur3e_wrist_1_link, child ur3e_wrist_2_link, origin xyz=0 -0.08535 -1.750557762378351e-11 rpy=1.570796327 0 0, axis 0 0 1, limit lower=-6.283185307179586 upper=6.283185307179586 effort=12.0 velocity=6.283185307179586
- added joint ur3e_wrist_3-flange: type fixed, parent ur3e_wrist_3_link, child ur3e_flange, origin xyz=0 0 0 rpy=0 -1.5707963267948966 -1.5707963267948966
- added joint ur3e_wrist_3_joint: type continuous, parent ur3e_wrist_2_link, child ur3e_wrist_3_link, origin xyz=0 0.0819 -1.679797079540562e-11 rpy=1.570796326589793 3.141592653589793 3.141592653589793, axis 0 0 1, limit effort=12.0 velocity=6.283185307179586
- added joint ur3e_wrist_3_link-ft_frame: type fixed, parent ur3e_wrist_3_link, child ur3e_ft_frame, origin xyz=0 0 0 rpy=3.141592653589793 0 0
